File: board/mainboard.sch (EAGLE design)
At the start: 10 parts, among them U1 DWM1000

Commit message: check dwm connections
Connections:
- removed net +12V: JP1.15
- removed net AREF: JP1.3
- removed net MLDIR: JP1.1
- removed net NRST: JP1.13
- removed net NRST1: JP2.3
- net GND: no longer JP2.4
Changed lines of the file:
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@@
 <part name="P+11" library="supply1" deviceset="+5V" device=""/>
 <part name="+3V5" library="supply1" deviceset="+3V3" device=""/>
-<part name="P+10" library="supply1" deviceset="+12V" device=""/>
 <part name="P+13" library="supply1" deviceset="+5V" device=""/>
 <part name="R1" library="rcl" deviceset="R-EU_" device="R0603" value="10k"/>
@@
 <instance part="P+11" gate="1" x="76.2" y="109.22"/>
 <instance part="+3V5" gate="G$1" x="78.74" y="63.5"/>
-<instance part="P+10" gate="1" x="152.4" y="63.5"/>
 <instance part="P+13" gate="1" x="160.02" y="63.5"/>
 <instance part="R1" gate="G$1" x="17.78" y="35.56" rot="R90"/>
@@
 <wire x1="147.32" y1="50.8" x2="152.4" y2="50.8" width="0.1524" layer="91"/>
 <label x="152.4" y="50.8" size="1.016" layer="95" xref="yes"/>
-</segment>
-<segment>
-<pinref part="JP2" gate="A" pin="4"/>
-<wire x1="129.54" y1="45.72" x2="116.84" y2="45.72" width="0.1524" layer="91"/>
-<label x="116.84" y="45.72" size="1.016" layer="95" rot="R180" xref="yes"/>
 </segment>
 <segment>
@@
 </segment>
 </net>
-<net name="+12V" class="0">
-<segment>
-<pinref part="JP1" gate="A" pin="15"/>
-<wire x1="147.32" y1="53.34" x2="152.4" y2="53.34" width="0.1524" layer="91"/>
-<label x="152.4" y="53.34" size="1.016" layer="95" xref="yes"/>
-<pinref part="P+10" gate="1" pin="+12V"/>
-<wire x1="152.4" y1="53.34" x2="152.4" y2="60.96" width="0.1524" layer="91"/>
-</segment>
-</net>
 <net name="+5V" class="0">
 <segment>
@@
 </segment>
 </net>
-<net name="NRST" class="0">
-<segment>
-<pinref part="JP1" gate="A" pin="13"/>
-<wire x1="147.32" y1="48.26" x2="152.4" y2="48.26" width="0.1524" layer="91"/>
-<label x="152.4" y="48.26" size="1.016" layer="95" xref="yes"/>
-</segment>
-</net>
 <net name="CSN" class="0">
 <segment>
@@
 </segment>
 </net>
-<net name="AREF" class="0">
-<segment>
-<pinref part="JP1" gate="A" pin="3"/>
-<wire x1="147.32" y1="22.86" x2="160.02" y2="22.86" width="0.1524" layer="91"/>
-<label x="160.02" y="22.86" size="1.016" layer="95" xref="yes"/>
-</segment>
-</net>
 <net name="SCK" class="0">
 <segment>
@@
 <wire x1="147.32" y1="35.56" x2="160.02" y2="35.56" width="0.1524" layer="91"/>
 <label x="160.02" y="35.56" size="1.016" layer="95" xref="yes"/>
-</segment>
-</net>
-<net name="NRST1" class="0">
-<segment>
-<pinref part="JP2" gate="A" pin="3"/>
-<wire x1="129.54" y1="48.26" x2="116.84" y2="48.26" width="0.1524" layer="91"/>
-<label x="116.84" y="48.26" size="1.016" layer="95" rot="R180" xref="yes"/>
 </segment>
 </net>
@@
 </segment>
 </net>
-<net name="MLDIR" class="0">
-<segment>
-<pinref part="JP1" gate="A" pin="1"/>
-<wire x1="147.32" y1="17.78" x2="160.02" y2="17.78" width="0.1524" layer="91"/>
-<label x="160.02" y="17.78" size="1.016" layer="95" xref="yes"/>
-</segment>
-</net>
