File: board/mainboard.sch (EAGLE design)
At the start: 10 parts, among them U1 DWM1000

Commit message: powerplug and mountings
Parts:
- removed C4: 100n, rcl:C-EUC0603K
- removed LED1: WS2812B, WS2812B:WS2812B
- added J1: 1X2-3.5MM, adafruit:1X2-3.5MM
Connections:
- net +5V: now also J1.1; no longer C4.1, LED1.VDD
- net GND: now also J1.2; no longer C4.2, LED1.GND
- net LED1: no longer LED1.DI
Changed lines of the file:
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@@
 <?xml version="1.0" encoding="utf-8"?>
 <!DOCTYPE eagle SYSTEM "eagle.dtd">
-<eagle version="7.7.0">
+<eagle version="7.1.0">
 <drawing>
 <settings>
@@
 <layers>
 <layer number="1" name="Top" color="4" fill="1" visible="no" active="no"/>
+<layer number="2" name="Route2" color="1" fill="3" visible="no" active="no"/>
+<layer number="3" name="Route3" color="4" fill="3" visible="no" active="no"/>
+<layer number="4" name="Route4" color="1" fill="4" visible="no" active="no"/>
+<layer number="5" name="Route5" color="4" fill="4" visible="no" active="no"/>
+<layer number="6" name="Route6" color="1" fill="8" visible="no" active="no"/>
+<layer number="7" name="Route7" color="4" fill="8" visible="no" active="no"/>
+<layer number="8" name="Route8" color="1" fill="2" visible="no" active="no"/>
+<layer number="9" name="Route9" color="4" fill="2" visible="no" active="no"/>
+<layer number="10" name="Route10" color="1" fill="7" visible="no" active="no"/>
+<layer number="11" name="Route11" color="4" fill="7" visible="no" active="no"/>
+<layer number="12" name="Route12" color="1" fill="5" visible="no" active="no"/>
+<layer number="13" name="Route13" color="4" fill="5" visible="no" active="no"/>
+<layer number="14" name="Route14" color="1" fill="6" visible="no" active="no"/>
+<layer number="15" name="Route15" color="4" fill="6" visible="no" active="no"/>
 <layer number="16" name="Bottom" color="1" fill="1" visible="no" active="no"/>
 <layer number="17" name="Pads" color="2" fill="1" visible="no" active="no"/>
@@
 <layer number="230" name="230bmp" color="7" fill="1" visible="yes" active="yes"/>
 <layer number="231" name="231bmp" color="7" fill="1" visible="yes" active="yes"/>
+<layer number="232" name="Eagle3D_PG2" color="7" fill="1" visible="no" active="no"/>
+<layer number="233" name="Eagle3D_PG3" color="7" fill="1" visible="no" active="no"/>
 <layer number="248" name="Housing" color="7" fill="1" visible="yes" active="yes"/>
 <layer number="249" name="Edge" color="7" fill="1" visible="yes" active="yes"/>
@@
 <parts>
 <part name="U1" library="DWM1000" deviceset="DWM1000" device=""/>
-<part name="LED1" library="WS2812B" deviceset="WS2812B" device=""/>
-<part name="C4" library="rcl" deviceset="C-EU" device="C0603K" value="100n"/>
 <part name="JP1" library="pinhead" deviceset="PINHD-1X15" device="" value="Nucleo R"/>
 <part name="JP2" library="pinhead" deviceset="PINHD-1X15" device="" value="Nucleo L"/>
 <part name="GND12" library="supply1" deviceset="GND" device=""/>
-<part name="GND13" library="supply1" deviceset="GND" device=""/>
-<part name="GND14" library="supply1" deviceset="GND" device=""/>
-<part name="P+11" library="supply1" deviceset="+5V" device=""/>
 <part name="+3V5" library="supply1" deviceset="+3V3" device=""/>
 <part name="P+13" library="supply1" deviceset="+5V" device=""/>
@@
 <part name="FRAME1" library="frames" deviceset="A4L-LOC" device=""/>
 <part name="+3V1" library="supply1" deviceset="+3V3" device=""/>
+<part name="J1" library="adafruit" deviceset="1X2" device="-3.5MM"/>
+<part name="GND2" library="supply1" deviceset="GND" device=""/>
+<part name="P+1" library="supply1" deviceset="+5V" device=""/>
 </parts>
 <sheets>
@@
 <instances>
 <instance part="U1" gate="G$1" x="53.34" y="38.1"/>
-<instance part="LED1" gate="G$1" x="99.06" y="93.98" rot="R90"/>
-<instance part="C4" gate="G$1" x="76.2" y="91.44"/>
 <instance part="JP1" gate="A" x="144.78" y="35.56" rot="R180"/>
 <instance part="JP2" gate="A" x="132.08" y="35.56"/>
 <instance part="GND12" gate="1" x="78.74" y="12.7"/>
-<instance part="GND13" gate="1" x="109.22" y="81.28"/>
-<instance part="GND14" gate="1" x="76.2" y="81.28"/>
-<instance part="P+11" gate="1" x="76.2" y="109.22"/>
 <instance part="+3V5" gate="G$1" x="78.74" y="63.5"/>
-<instance part="P+13" gate="1" x="160.02" y="63.5"/>
+<instance part="P+13" gate="1" x="160.02" y="58.42"/>
 <instance part="R1" gate="G$1" x="17.78" y="35.56" rot="R90"/>
 <instance part="R2" gate="G$1" x="22.86" y="20.32" rot="R90"/>
@@
 <instance part="FRAME1" gate="G$1" x="-33.02" y="-40.64"/>
 <instance part="+3V1" gate="G$1" x="172.72" y="25.4"/>
+<instance part="J1" gate="G$1" x="109.22" y="7.62" rot="R90"/>
+<instance part="GND2" gate="1" x="109.22" y="-5.08"/>
+<instance part="P+1" gate="1" x="99.06" y="7.62"/>
 </instances>
 <busses>
@@
 </segment>
 <segment>
-<pinref part="C4" gate="G$1" pin="2"/>
-<pinref part="GND14" gate="1" pin="GND"/>
-<wire x1="76.2" y1="83.82" x2="76.2" y2="86.36" width="0.1524" layer="91"/>
-</segment>
-<segment>
-<pinref part="LED1" gate="G$1" pin="GND"/>
-<pinref part="GND13" gate="1" pin="GND"/>
-<wire x1="109.22" y1="93.98" x2="109.22" y2="83.82" width="0.1524" layer="91"/>
-</segment>
-<segment>
 <pinref part="R1" gate="G$1" pin="1"/>
 <pinref part="GND1" gate="1" pin="GND"/>
@@
 <junction x="25.4" y="2.54"/>
 </segment>
+<segment>
+<pinref part="J1" gate="G$1" pin="2"/>
+<wire x1="109.22" y1="2.54" x2="109.22" y2="-2.54" width="0.1524" layer="91"/>
+<pinref part="GND2" gate="1" pin="GND"/>
+</segment>
 </net>
 <net name="+5V" class="0">
-<segment>
-<pinref part="LED1" gate="G$1" pin="VDD"/>
-<pinref part="C4" gate="G$1" pin="1"/>
-<wire x1="83.82" y1="93.98" x2="76.2" y2="93.98" width="0.1524" layer="91"/>
-<pinref part="P+11" gate="1" pin="+5V"/>
-<wire x1="76.2" y1="93.98" x2="76.2" y2="106.68" width="0.1524" layer="91"/>
-<junction x="76.2" y="93.98"/>
-</segment>
 <segment>
 <pinref part="JP1" gate="A" pin="12"/>
@@
 <label x="160.02" y="45.72" size="1.016" layer="95" xref="yes"/>
 <pinref part="P+13" gate="1" pin="+5V"/>
-<wire x1="160.02" y1="45.72" x2="160.02" y2="60.96" width="0.1524" layer="91"/>
+<wire x1="160.02" y1="45.72" x2="160.02" y2="55.88" width="0.1524" layer="91"/>
+</segment>
+<segment>
+<pinref part="J1" gate="G$1" pin="1"/>
+<wire x1="106.68" y1="2.54" x2="106.68" y2="-2.54" width="0.1524" layer="91"/>
+<wire x1="106.68" y1="-2.54" x2="99.06" y2="-2.54" width="0.1524" layer="91"/>
+<wire x1="99.06" y1="-2.54" x2="99.06" y2="5.08" width="0.1524" layer="91"/>
+<pinref part="P+1" gate="1" pin="+5V"/>
 </segment>
 </net>
 <net name="LED1" class="0">
 <segment>
-<pinref part="LED1" gate="G$1" pin="DI"/>
-<wire x1="101.6" y1="81.28" x2="101.6" y2="76.2" width="0.1524" layer="91"/>
-<wire x1="101.6" y1="76.2" x2="116.84" y2="76.2" width="0.1524" layer="91"/>
-<label x="116.84" y="76.2" size="1.778" layer="95" xref="yes"/>
-</segment>
-<segment>
 <pinref part="JP2" gate="A" pin="5"/>
